Commit message: Support alternative differential steering mode

File: urdf/controllers/diff_drive.urdf.xacro (robot description, xacro)
@@ -1,10 +1,8 @@
 <robot xmlns:xacro="http://ros.org/wiki/xacro">
-  <xacro:macro name="diff_drive_controller" params="wheel_separation wheel_radius wheel_torque">
+  <xacro:macro name="diff_drive_controller" params="wheel_separation wheel_radius wheel_torque gz_odom_topic gz_cmd_vel_topic">
     <gazebo>
-      <plugin
-        filename="gz-sim-diff-drive-system"
-        name="gz::sim::systems::DiffDrive">
-        <left_joint>left_wheel_joint</left_joint>
-        <right_joint>right_wheel_joint</right_joint>
+      <plugin filename="gz-sim-diff-drive-system" name="gz::sim::systems::DiffDrive">
+        <left_joint>rear_left_wheel_joint</left_joint>
+        <right_joint>rear_right_wheel_joint</right_joint>
         <wheel_separation>${wheel_separation}</wheel_separation>
         <wheel_radius>${wheel_radius * 2}</wheel_radius>
@@ -17,13 +15,13 @@
         <max_angular_velocity>1</max_angular_velocity>
         <min_angular_velocity>-1</min_angular_velocity>
-        <topic>cmd_vel</topic>
-        <odom_topic>odom</odom_topic>
+        <odom_topic>${gz_odom_topic}</odom_topic>
         <odom_publish_frequency>20</odom_publish_frequency>
+        <topic>${gz_cmd_vel_topic}</topic>
         <frame_id>odom</frame_id>
         <child_frame_id>base_footprint</child_frame_id>
       </plugin>
       <plugin filename="gz-sim-joint-state-publisher-system" name="gz::sim::systems::JointStatePublisher">
-        <joint_name>left_wheel_joint</joint_name>
-        <joint_name>front_right_wheel_joint</joint_name>
+        <joint_name>rear_left_wheel_joint</joint_name>
+        <joint_name>rear_right_wheel_joint</joint_name>
         <topic>/joint_states</topic>
       </plugin>

File: urdf/mech/base.urdf.xacro (robot description, xacro)
@@ -41,5 +41,5 @@
       <parent link="base_footprint"/>
       <child link="base_link"/>
-      <origin xyz="${-base_link_x_offset_to_center} 0 ${wheel_radius + -1*wheel_pos_z - base_link_z_offset_to_center}" rpy="0 0 0"/>
+      <origin xyz="0 0 ${wheel_radius + -1*wheel_pos_z - base_link_z_offset_to_center}" rpy="0 0 0"/>
     </joint>
   </xacro:macro>

File: urdf/robots/ebot_2wd_common.urdf.xacro (robot description, xacro)
@@ -1,13 +1,9 @@
 <?xml version="1.0"?>
 <robot name="elsabot_robot" xmlns:xacro="http://ros.org/wiki/xacro">
-  <xacro:include filename="$(find elsabot_robot)/urdf/2wd_properties.urdf.xacro" />
   <xacro:include filename="$(find elsabot_robot)/urdf/mech/base.urdf.xacro" />
-  <xacro:include filename="$(find elsabot_robot)/urdf/mech/wheel.urdf.xacro" />
-  <xacro:include filename="$(find elsabot_robot)/urdf/mech/wheel_steering.urdf.xacro" />
   <xacro:include filename="$(find elsabot_robot)/urdf/sensors/imu.urdf.xacro" />
   <xacro:include filename="$(find elsabot_robot)/urdf/sensors/gps.urdf.xacro" />
   <xacro:include filename="$(find elsabot_robot)/urdf/sensors/generic_laser.urdf.xacro" />
   <xacro:include filename="$(find elsabot_robot)/urdf/sensors/oakd_on_ptbase.urdf.xacro" />
-  <xacro:include filename="$(find elsabot_robot)/urdf/controllers/ackermann_drive.urdf.xacro" />
   <xacro:include filename="$(find elsabot_robot)/urdf/sensors/hcsr04.urdf.xacro" />
   <xacro:include filename="$(find elsabot_robot)/urdf/sensors/hcsr04_servo_pan_mount.xacro" />
@@ -20,62 +16,4 @@
     wheel_pos_z="${wheel_pos_z}"
     mesh="package://elsabot_robot/meshes/ebot.stl"
-  />
-  <xacro:wheel
-    parent_link="front_left_wheel_steering_link"
-    side="front_left"
-    radius="${wheel_radius}"
-    width="${wheel_width}"
-    pos_x="0"
-    pos_y="${wheel_center_to_kingpin}"
-    pos_z="0"
-    mass="${wheel_mass}"
-  />
-  <xacro:wheel
-    parent_link="front_right_wheel_steering_link"
-    side="front_right"
-    radius="${wheel_radius}"
-    width="${wheel_width}"
-    pos_x="0"
-    pos_y="${-wheel_center_to_kingpin}"
-    pos_z="0"
-    mass="${wheel_mass}"
-  />
-  <xacro:wheel
-    parent_link="base_link"
-    side="rear_left"
-    radius="${wheel_radius}"
-    width="${wheel_width}"
-    pos_x="${-wheel_pos_x_rear + base_link_x_offset_to_center}"
-    pos_y="${wheel_pos_y}"
-    pos_z="${wheel_pos_z + base_link_z_offset_to_center}"
-    mass="${wheel_mass}"
-  />
-  <xacro:wheel
-    parent_link="base_link"
-    side="rear_right"
-    radius="${wheel_radius}"
-    width="${wheel_width}"
-    pos_x="${-wheel_pos_x_rear + base_link_x_offset_to_center}"
-    pos_y="${-wheel_pos_y}"
-    pos_z="${wheel_pos_z + base_link_z_offset_to_center}"
-    mass="${wheel_mass}"
-  />
-  <xacro:wheel_steering
-    parent_link="base_link"
-    side="front_left"
-    pos_x="${wheel_pos_x_front + base_link_x_offset_to_center}"
-    pos_y="${kingpin_width/2}"
-    pos_z="${wheel_pos_z + base_link_z_offset_to_center}"
-    mass="${wheel_mass_steering}"
-    max_steer="${wheel_max_steer}"
-  />
-  <xacro:wheel_steering
-    parent_link="base_link"
-    side="front_right"
-    pos_x="${wheel_pos_x_front + base_link_x_offset_to_center}"
-    pos_y="${-kingpin_width/2}"
-    pos_z="${wheel_pos_z + base_link_z_offset_to_center}"
-    mass="${wheel_mass_steering}"
-    max_steer="${wheel_max_steer}"
   />
   <xacro:generic_laser
@@ -127,12 +65,3 @@
     <plugin filename="gz-sim-navsat-system" name="gz::sim::systems::NavSat"/>
   </gazebo>
-  <xacro:ackermann_drive_controller
-    wheel_base = "${wheel_base}"
-    wheel_max_steer = "${wheel_max_steer}"
-    wheel_separation = "${2*wheel_pos_y}"
-    kingpin_width = "${kingpin_width}"
-    wheel_radius = "${wheel_radius}"
-    gz_odom_topic="/ebot/odom"
-    gz_cmd_vel_topic="/cmd_vel/muxed"
-  />
 </robot>
