Commit message: Changes for Gazebo support

File: urdf/2wd_properties.urdf.xacro (robot description, xacro)
@@ -5,5 +5,5 @@
   <xacro:property name="base_width" value="0.483" />
   <xacro:property name="base_height" value="0.365" />
-  <xacro:property name="base_mass" value="10" />
+  <xacro:property name="base_mass" value="18" />
   <xacro:property name="wheel_base" value="0.368" />
   <xacro:property name="wheel_radius" value="0.08" />

File: urdf/robots/ebot_2wd.urdf.xacro (robot description, xacro)
@@ -110,5 +110,5 @@
     wheel_radius = "${wheel_radius}"
     gz_odom_topic="/ebot/odom"
-    gz_cmd_vel_topic="cmd_vel"
+    gz_cmd_vel_topic="/cmd_vel/muxed"
   />
 </robot>

Commit message: Adjust lidar position for new mounting position

File: urdf/2wd_properties.urdf.xacro (robot description, xacro)
@@ -24,5 +24,5 @@
   <xacro:property name="base_link_z_offset_to_center" value="${-1*wheel_pos_z}" />
   <xacro:property name="laser_pose">
-    <origin xyz="${0.205 + base_link_x_offset_to_center} 0 ${0.092 + base_link_z_offset_to_center}" rpy="0 0 3.14"/>
+    <origin xyz="${-0.01 + base_link_x_offset_to_center} 0 ${0.35 + base_link_z_offset_to_center}" rpy="0 0 3.14"/>
   </xacro:property>
   <xacro:property name="imu_pose">

Commit message: Support HCSR04 sensors on servo mount
New front and back HCSR04 sensors mounted on servo for panning left and right.

File: urdf/2wd_properties.urdf.xacro (robot description, xacro)
@@ -35,3 +35,15 @@
     <origin xyz="${-0.030  + base_link_x_offset_to_center} 0 ${0.535 + base_link_z_offset_to_center}" rpy="0 0 0"/>
   </xacro:property>
+  <xacro:property name="hcsr04_range_front_servo_pose">
+    <origin xyz="${0.245 + base_link_x_offset_to_center} 0.0 ${-0.070 + base_link_z_offset_to_center}" rpy="0 0 0"/>
+  </xacro:property>
+  <xacro:property name="hcsr04_range_front_pose">
+    <origin xyz="0.010 0.0 0.0" rpy="0 0 0"/>
+  </xacro:property>
+  <xacro:property name="hcsr04_range_back_servo_pose">
+    <origin xyz="${-0.254 + base_link_x_offset_to_center} 0.053 ${-0.070 + base_link_z_offset_to_center}" rpy="0 0 -3.14"/>
+  </xacro:property>
+  <xacro:property name="hcsr04_range_back_pose">
+    <origin xyz="-0.020 0.0 0.0" rpy="0 0 0"/>
+  </xacro:property>
 </robot>

File: urdf/robots/ebot_2wd.urdf.xacro (robot description, xacro)
@@ -10,4 +10,6 @@
   <xacro:include filename="$(find elsabot_robot)/urdf/sensors/oakd_on_ptbase.urdf.xacro" />
   <xacro:include filename="$(find elsabot_robot)/urdf/controllers/ackermann_drive.urdf.xacro" />
+  <xacro:include filename="$(find elsabot_robot)/urdf/sensors/hcsr04.urdf.xacro" />
+  <xacro:include filename="$(find elsabot_robot)/urdf/sensors/hcsr04_servo_pan_mount.xacro" />
   <xacro:base
     length="${base_length}"
@@ -94,4 +96,26 @@
     <xacro:insert_block name="depth_sensor_pose" />
   </xacro:depth_sensor>
+  <xacro:hcsr04_servo_pan_mount
+    frame_id="hcsr04_pan_joint_front"
+    parent_link="base_link"
+    child_link="hcsr04_front_servo_pan_link">
+    <xacro:insert_block name="hcsr04_range_front_servo_pose" />
+  </xacro:hcsr04_servo_pan_mount>
+  <xacro:hcsr04_sensor
+    frame_id="hcsr04_front"
+    parent_link="hcsr04_front_servo_pan_link">
+    <xacro:insert_block name="hcsr04_range_front_pose" />
+  </xacro:hcsr04_sensor>
+  <xacro:hcsr04_servo_pan_mount
+    frame_id="hcsr04_pan_joint_back"
+    parent_link="base_link"
+    child_link="hcsr04_back_servo_pan_link">
+    <xacro:insert_block name="hcsr04_range_back_servo_pose" />
+  </xacro:hcsr04_servo_pan_mount>
+  <xacro:hcsr04_sensor
+    frame_id="hcsr04_back"
+    parent_link="hcsr04_back_servo_pan_link">
+    <xacro:insert_block name="hcsr04_range_back_pose" />
+  </xacro:hcsr04_sensor>
   <gazebo>
     <plugin filename="gz-sim-joint-state-publisher-system" name="gz::sim::systems::JointStatePublisher"/>

File: urdf/sensors/hcsr04.urdf.xacro (robot description, xacro)
@@ -1,5 +1,5 @@
 <robot xmlns:xacro="http://ros.org/wiki/xacro">
   <xacro:property name="M_PI" value="3.1415926535897931" />
-    <xacro:macro name="hcsr04_sensor" params="*origin frame_id">
+    <xacro:macro name="hcsr04_sensor" params="*origin frame_id parent_link">
       <link name="${frame_id}">
         <inertial>
@@ -17,5 +17,5 @@
       <joint name="${frame_id}_joint" type="fixed">
         <xacro:insert_block name="origin" />
-        <parent link="base_link" />
+        <parent link="${parent_link}" />
         <child link="${frame_id}"/>
       </joint>

Commit message: Testing new location of imu to avoid interference.

File: urdf/2wd_properties.urdf.xacro (robot description, xacro)
@@ -27,5 +27,5 @@
   </xacro:property>
   <xacro:property name="imu_pose">
-    <origin xyz="${0.020 + base_link_x_offset_to_center} 0.0 ${0.220 + base_link_z_offset_to_center}" rpy="0 0 0"/>
+    <origin xyz="${-0.245 + base_link_x_offset_to_center} 0.0 ${0.145 + base_link_z_offset_to_center}" rpy="0 0 0"/>
   </xacro:property>
   <xacro:property name="gps_pose">

Commit message: Testing new location of imu to avoid interference.

File: urdf/2wd_properties.urdf.xacro (robot description, xacro)
@@ -27,5 +27,5 @@
   </xacro:property>
   <xacro:property name="imu_pose">
-    <origin xyz="${-0.245 + base_link_x_offset_to_center} 0.0 ${0.145 + base_link_z_offset_to_center}" rpy="0 0 0"/>
+    <origin xyz="${-0.105 + base_link_x_offset_to_center} -0.065 ${0.436 + base_link_z_offset_to_center}" rpy="0 0 0"/>
   </xacro:property>
   <xacro:property name="gps_pose">

Commit message: Add support for two V53L7CX TOF sensors on front.

File: urdf/2wd_properties.urdf.xacro (robot description, xacro)
@@ -1,4 +1,5 @@
 <?xml version="1.0"?>
 <robot xmlns:xacro="http://ros.org/wiki/xacro">
+  <xacro:property name="M_PI" value="3.1415926535897931" />
   <!-- x,y positions are relative to the center of the robot -->
   <xacro:property name="base_length" value="0.525" />
@@ -24,5 +25,5 @@
   <xacro:property name="base_link_z_offset_to_center" value="${-1*wheel_pos_z}" />
   <xacro:property name="laser_pose">
-    <origin xyz="${-0.01 + base_link_x_offset_to_center} 0 ${0.35 + base_link_z_offset_to_center}" rpy="0 0 3.14"/>
+    <origin xyz="${-0.01 + base_link_x_offset_to_center} 0 ${0.35 + base_link_z_offset_to_center}" rpy="0 0 ${M_PI}"/>
   </xacro:property>
   <xacro:property name="imu_pose">
@@ -33,5 +34,5 @@
   </xacro:property>
   <xacro:property name="depth_sensor_pose">
-    <origin xyz="${-0.030  + base_link_x_offset_to_center} 0 ${0.535 + base_link_z_offset_to_center}" rpy="0 0 0"/>
+    <origin xyz="${-0.030 + base_link_x_offset_to_center} 0 ${0.535 + base_link_z_offset_to_center}" rpy="0 0 0"/>
   </xacro:property>
   <xacro:property name="hcsr04_range_front_servo_pose">
@@ -42,8 +43,20 @@
   </xacro:property>
   <xacro:property name="hcsr04_range_back_servo_pose">
-    <origin xyz="${-0.254 + base_link_x_offset_to_center} 0.053 ${-0.070 + base_link_z_offset_to_center}" rpy="0 0 -3.14"/>
+    <origin xyz="${-0.254 + base_link_x_offset_to_center} 0.053 ${-0.070 + base_link_z_offset_to_center}" rpy="0 0 -${M_PI}"/>
   </xacro:property>
   <xacro:property name="hcsr04_range_back_pose">
     <origin xyz="-0.020 0.0 0.0" rpy="0 0 0"/>
   </xacro:property>
+  <xacro:property name="tof_front_stepper_pose">
+    <origin xyz="${0.245 + base_link_x_offset_to_center} 0.0 ${-0.070 + base_link_z_offset_to_center}" rpy="0 0 0"/>
+  </xacro:property>
+  <xacro:property name="tof_sensor_front_pose">
+    <origin xyz="0.0 0.0 0.0" rpy="0 0 0"/>
+  </xacro:property>
+  <xacro:property name="tof_sensor_front_left_pose">
+    <origin xyz="${0.240 + base_link_x_offset_to_center} 0.013 ${-0.038 + base_link_z_offset_to_center}" rpy="0 0 ${M_PI*30.0/180.0}"/>
+  </xacro:property>
+  <xacro:property name="tof_sensor_front_right_pose">
+    <origin xyz="${0.240 + base_link_x_offset_to_center} -0.013 ${-0.038 + base_link_z_offset_to_center}" rpy="0 0 -${M_PI*30.0/180.0}"/>
+  </xacro:property>
 </robot>

File: urdf/robots/ebot_2wd_common.urdf.xacro (robot description, xacro)
@@ -8,4 +8,6 @@
   <xacro:include filename="$(find elsabot_robot)/urdf/sensors/hcsr04.urdf.xacro" />
   <xacro:include filename="$(find elsabot_robot)/urdf/sensors/hcsr04_servo_pan_mount.xacro" />
+  <xacro:include filename="$(find elsabot_robot)/urdf/sensors/tof.urdf.xacro" />
+  <xacro:include filename="$(find elsabot_robot)/urdf/sensors/tof_stepper_pan_mount.xacro" />
   <xacro:base
     length="${base_length}"
@@ -56,4 +58,26 @@
     <xacro:insert_block name="hcsr04_range_back_pose" />
   </xacro:hcsr04_sensor>
+  <!-- TOF on stepper not used -->
+  <!--xacro:tof_stepper_pan_mount
+    frame_id="tof_pan_joint_front"
+    parent_link="base_link"
+    child_link="tof_front_stepper_servo_pan_link">
+    <xacro:insert_block name="tof_front_stepper_pose" />
+  </xacro:tof_stepper_pan_mount-->
+  <!--xacro:tof_sensor
+    frame_id="front_tof_frame"
+    parent_link="tof_front_stepper_servo_pan_link">
+    <xacro:insert_block name="tof_sensor_front_pose" />
+  </xacro:tof_sensor-->
+  <xacro:tof_sensor
+    frame_id="front_left_tof_frame"
+    parent_link="base_link">
+    <xacro:insert_block name="tof_sensor_front_left_pose" />
+  </xacro:tof_sensor>
+<xacro:tof_sensor
+    frame_id="front_right_tof_frame"
+    parent_link="base_link">
+    <xacro:insert_block name="tof_sensor_front_right_pose" />
+  </xacro:tof_sensor>
   <gazebo>
     <plugin filename="gz-sim-joint-state-publisher-system" name="gz::sim::systems::JointStatePublisher"/>
