Commit message: Add suport for rear vl53l7cx TOF sensors

File: urdf/2wd_properties.urdf.xacro (robot description, xacro)
@@ -60,3 +60,9 @@
     <origin xyz="${0.240 + base_link_x_offset_to_center} -0.013 ${-0.038 + base_link_z_offset_to_center}" rpy="0 0 -${M_PI*30.0/180.0}"/>
   </xacro:property>
+  <xacro:property name="tof_sensor_back_left_pose">
+    <origin xyz="${-0.235 + base_link_x_offset_to_center} ${0.013-0.044} ${-0.038 + base_link_z_offset_to_center}" rpy="0 0 ${M_PI*(180.0-30.0)/180.0}"/>
+  </xacro:property>
+  <xacro:property name="tof_sensor_back_right_pose">
+    <origin xyz="${-0.235 + base_link_x_offset_to_center} ${-0.013-0.044} ${-0.038 + base_link_z_offset_to_center}" rpy="0 0 -${M_PI*(180.0-30.0)/180.0}"/>
+  </xacro:property>
 </robot>

File: urdf/robots/ebot_2wd_common.urdf.xacro (robot description, xacro)
@@ -10,4 +10,8 @@
   <xacro:include filename="$(find elsabot_robot)/urdf/sensors/tof.urdf.xacro" />
   <xacro:include filename="$(find elsabot_robot)/urdf/sensors/tof_stepper_pan_mount.xacro" />
+  <!-- Set to true of if using an hcsr04 on a panning servo base -->
+  <xacro:property name="use_hcsr04" value="false" />
+  <!-- Set to true of TOF sensor mounted on panning stepper base -->
+  <xacro:property name="use_rotating_tof" value="false" />
   <xacro:base
     length="${base_length}"
@@ -36,48 +40,63 @@
     <xacro:insert_block name="depth_sensor_pose" />
   </xacro:depth_sensor>
-  <xacro:hcsr04_servo_pan_mount
-    frame_id="hcsr04_pan_joint_front"
-    parent_link="base_link"
-    child_link="hcsr04_front_servo_pan_link">
-    <xacro:insert_block name="hcsr04_range_front_servo_pose" />
-  </xacro:hcsr04_servo_pan_mount>
-  <xacro:hcsr04_sensor
-    frame_id="hcsr04_front"
-    parent_link="hcsr04_front_servo_pan_link">
-    <xacro:insert_block name="hcsr04_range_front_pose" />
-  </xacro:hcsr04_sensor>
-  <xacro:hcsr04_servo_pan_mount
-    frame_id="hcsr04_pan_joint_back"
-    parent_link="base_link"
-    child_link="hcsr04_back_servo_pan_link">
-    <xacro:insert_block name="hcsr04_range_back_servo_pose" />
-  </xacro:hcsr04_servo_pan_mount>
-  <xacro:hcsr04_sensor
-    frame_id="hcsr04_back"
-    parent_link="hcsr04_back_servo_pan_link">
-    <xacro:insert_block name="hcsr04_range_back_pose" />
-  </xacro:hcsr04_sensor>
-  <!-- TOF on stepper not used -->
-  <!--xacro:tof_stepper_pan_mount
-    frame_id="tof_pan_joint_front"
-    parent_link="base_link"
-    child_link="tof_front_stepper_servo_pan_link">
-    <xacro:insert_block name="tof_front_stepper_pose" />
-  </xacro:tof_stepper_pan_mount-->
-  <!--xacro:tof_sensor
-    frame_id="front_tof_frame"
-    parent_link="tof_front_stepper_servo_pan_link">
-    <xacro:insert_block name="tof_sensor_front_pose" />
-  </xacro:tof_sensor-->
-  <xacro:tof_sensor
-    frame_id="front_left_tof_frame"
-    parent_link="base_link">
-    <xacro:insert_block name="tof_sensor_front_left_pose" />
-  </xacro:tof_sensor>
-<xacro:tof_sensor
-    frame_id="front_right_tof_frame"
-    parent_link="base_link">
-    <xacro:insert_block name="tof_sensor_front_right_pose" />
-  </xacro:tof_sensor>
+  <xacro:if value="${use_hcsr04}">
+    <xacro:hcsr04_servo_pan_mount
+      frame_id="hcsr04_pan_joint_front"
+      parent_link="base_link"
+      child_link="hcsr04_front_servo_pan_link">
+      <xacro:insert_block name="hcsr04_range_front_servo_pose" />
+    </xacro:hcsr04_servo_pan_mount>
+    <xacro:hcsr04_sensor
+      frame_id="hcsr04_front"
+      parent_link="hcsr04_front_servo_pan_link">
+      <xacro:insert_block name="hcsr04_range_front_pose" />
+    </xacro:hcsr04_sensor>
+    <xacro:hcsr04_servo_pan_mount
+      frame_id="hcsr04_pan_joint_back"
+      parent_link="base_link"
+      child_link="hcsr04_back_servo_pan_link">
+      <xacro:insert_block name="hcsr04_range_back_servo_pose" />
+    </xacro:hcsr04_servo_pan_mount>
+    <xacro:hcsr04_sensor
+      frame_id="hcsr04_back"
+      parent_link="hcsr04_back_servo_pan_link">
+      <xacro:insert_block name="hcsr04_range_back_pose" />
+    </xacro:hcsr04_sensor>
+  </xacro:if>
+  <xacro:if value="${use_rotating_tof}">
+    <xacro:tof_stepper_pan_mount
+      frame_id="tof_pan_joint_front"
+      parent_link="base_link"
+      child_link="tof_front_stepper_servo_pan_link">
+      <xacro:insert_block name="tof_front_stepper_pose" />
+    </xacro:tof_stepper_pan_mount>
+    <xacro:tof_sensor
+      frame_id="front_tof_frame"
+      parent_link="tof_front_stepper_servo_pan_link">
+      <xacro:insert_block name="tof_sensor_front_pose" />
+    </xacro:tof_sensor>
+  </xacro:if>
+  <xacro:unless value="${use_rotating_tof}">
+    <xacro:tof_sensor
+      frame_id="front_left_tof_frame"
+      parent_link="base_link">
+      <xacro:insert_block name="tof_sensor_front_left_pose" />
+    </xacro:tof_sensor>
+    <xacro:tof_sensor
+      frame_id="front_right_tof_frame"
+      parent_link="base_link">
+      <xacro:insert_block name="tof_sensor_front_right_pose" />
+    </xacro:tof_sensor>
+    <xacro:tof_sensor
+      frame_id="back_left_tof_frame"
+      parent_link="base_link">
+      <xacro:insert_block name="tof_sensor_back_left_pose" />
+    </xacro:tof_sensor>
+    <xacro:tof_sensor
+      frame_id="back_right_tof_frame"
+      parent_link="base_link">
+      <xacro:insert_block name="tof_sensor_back_right_pose" />
+    </xacro:tof_sensor>
+  </xacro:unless>
   <gazebo>
     <plugin filename="gz-sim-joint-state-publisher-system" name="gz::sim::systems::JointStatePublisher"/>

Commit message: Moved IMU sensor

File: urdf/2wd_properties.urdf.xacro (robot description, xacro)
@@ -28,5 +28,5 @@
   </xacro:property>
   <xacro:property name="imu_pose">
-    <origin xyz="${-0.105 + base_link_x_offset_to_center} -0.065 ${0.436 + base_link_z_offset_to_center}" rpy="0 0 0"/>
+    <origin xyz="${0.043 + base_link_x_offset_to_center} -0.096 ${0.330 + base_link_z_offset_to_center}" rpy="0 0 0"/>
   </xacro:property>
   <xacro:property name="gps_pose">
