Commit message: Jeep related support

File: urdf/jeep_properties.urdf.xacro (robot description, xacro)
@@ -1,5 +1,9 @@
 <?xml version="1.0"?>
 <robot xmlns:xacro="http://ros.org/wiki/xacro">
-  <xacro:property name="base_length" value="0.110" />
+  <xacro:property name="M_PI" value="3.1415926535897931" />
+  <!-- x,y positions are relative to the center of the robot -->
+  <!-- Set to true of if using an IMU mounted on the base -->
+  <xacro:property name="use_base_imu" value="false" />
+  <xacro:property name="base_length" value="01.10" />
   <xacro:property name="base_width" value="0.653" />
   <xacro:property name="base_height" value="0.450" />
@@ -8,5 +12,6 @@
   <xacro:property name="wheel_radius" value="0.140" />
   <xacro:property name="wheel_width" value="0.170" />
-  <xacro:property name="wheel_pos_x" value="0.354" />
+  <xacro:property name="wheel_pos_x_rear" value="-0.354" />
+  <xacro:property name="wheel_pos_x_front" value="0.354" />
   <xacro:property name="wheel_pos_y" value="0.3265" />
   <xacro:property name="wheel_pos_z" value="0.0" />
@@ -17,29 +22,41 @@
   <xacro:property name="kingpin_width" value="0.490" />
   <xacro:property name="wheel_center_to_kingpin" value="0.082" />
+  <!-- base_link_*_offset_to_center is used to move the base link x,z
+       origin to the rear axle center when using ackermann steering. -->
+  <xacro:property name="base_link_x_offset_to_center" value="${-wheel_pos_x_rear}" />
+  <xacro:property name="base_link_z_offset_to_center" value="0.0" />
   <xacro:property name="laser_pose">
-    <origin xyz="0.354 0 0.440" rpy="0 0 3.14"/>
+    <origin xyz="${0.354 + base_link_x_offset_to_center} 0 ${0.440 + base_link_z_offset_to_center}" rpy="0 0 3.14"/>
   </xacro:property>
-  <xacro:property name="imu_pose">
-    <origin xyz="-0.331 0.055 0.066" rpy="0 0 0"/>
+  <!-- IMU mounted on base -->
+  <xacro:if value="${use_base_imu}">
+    <xacro:property name="imu_pose">
+      <origin xyz="${-0.331 + base_link_x_offset_to_center} 0.055 ${0.066 + base_link_z_offset_to_center}" rpy="0 0 0"/>
+    </xacro:property>
+  </xacro:if>
+  <!-- IMU mounted on vertical rack -->
+  <xacro:unless value="${use_base_imu}">
+    <xacro:property name="imu_pose">
+      <origin xyz="${-0.504 + 0.02 + base_link_x_offset_to_center} -0.095 ${0.298 + 0.340 + base_link_z_offset_to_center}" rpy="0 0 0"/>
+    </xacro:property>
+  </xacro:unless>
+  <xacro:property name="gps_pose">
+    <origin xyz="${-0.504 - 0.150 + base_link_x_offset_to_center} 0.0 ${0.298 + 0.7 + base_link_z_offset_to_center}" rpy="0 0 0" />
   </xacro:property>
   <xacro:property name="depth_sensor_pose">
-    <origin xyz="-0.065 0 0.255" rpy="0 0 0"/>
+    <origin xyz="${-0.504 + 0.01 + base_link_x_offset_to_center} 0 ${0.298 + 0.540 + base_link_z_offset_to_center}" rpy="0 0 0"/>
   </xacro:property>
-  <xacro:property name="range_back_left_pose">
-    <origin xyz="-0.543 0.205 0.298" rpy="0 0 -3.14"/>
+  <xacro:property name="hcsr04_range_back_left_pose">
+    <origin xyz="${-0.543 + base_link_x_offset_to_center} 0.205 ${0.298 + base_link_z_offset_to_center}" rpy="0 0 -3.14"/>
   </xacro:property>
-  <xacro:property name="range_back_right_pose">
-    <origin xyz="-0.543 -0.205 0.298" rpy="0 0 -3.14"/>
+  <xacro:property name="hcsr04_range_back_right_pose">
+    <origin xyz="${-0.543 + base_link_x_offset_to_center} -0.205 ${0.298 + base_link_z_offset_to_center}" rpy="0 0 -3.14"/>
   </xacro:property>
-  <!-- OakD as depth sensor -->
-  <xacro:property name="depth_camera_name" value="oak" />
-  <xacro:property name="depth_camera_model" value="OAK-D" />
-  <xacro:property name="depth_base_frame" value="front_oakd_base_link" />
-  <xacro:property name="depth_parent_frame" value="base_link" />
-  <xacro:property name="depth_cam_pos_x" value="0.254" />
-  <xacro:property name="depth_cam_pos_y" value="0.0" />
-  <xacro:property name="depth_cam_pos_z" value="0.620" />
-  <xacro:property name="depth_cam_roll" value="0.0" />
-  <xacro:property name="depth_cam_pitch" value="0.42" />
-  <xacro:property name="depth_cam_yaw" value="0.0" />
+  <!-- Fix - check pitch angle and y offset -->
+  <xacro:property name="tof_sensor_front_left_pose">
+    <origin xyz="${0.530 + base_link_x_offset_to_center} 0.013 ${0.095 + base_link_z_offset_to_center}" rpy="0 ${M_PI*12.0/180.0} ${M_PI*30.0/180.0}"/>
+  </xacro:property>
+  <xacro:property name="tof_sensor_front_right_pose">
+    <origin xyz="${0.530 + base_link_x_offset_to_center} -0.013 ${0.095 + base_link_z_offset_to_center}" rpy="0 ${M_PI*12.0/180.0} -${M_PI*30.0/180.0}"/>
+  </xacro:property>
 </robot>

File: urdf/robots/jeep.urdf.xacro (robot description, xacro)
@@ -6,10 +6,10 @@
   <xacro:include filename="$(find elsabot_robot)/urdf/mech/wheel_steering.urdf.xacro" />
   <xacro:include filename="$(find elsabot_robot)/urdf/sensors/imu.urdf.xacro" />
+  <xacro:include filename="$(find elsabot_robot)/urdf/sensors/gps.urdf.xacro" />
   <xacro:include filename="$(find elsabot_robot)/urdf/sensors/generic_laser.urdf.xacro" />
-  <xacro:include filename="$(find elsabot_robot)/urdf/sensors/depthai_macro.urdf.xacro" />
   <xacro:include filename="$(find elsabot_robot)/urdf/sensors/oakd_on_ptbase.urdf.xacro" />
   <xacro:include filename="$(find elsabot_robot)/urdf/sensors/hcsr04.urdf.xacro" />
+  <xacro:include filename="$(find elsabot_robot)/urdf/sensors/tof.urdf.xacro" />
   <xacro:include filename="$(find elsabot_robot)/urdf/controllers/ackermann_drive.urdf.xacro" />
-  <!--xacro:include filename="$(find elsabot_robot)/urdf/sensors/depth_sensor.urdf.xacro" /-->
   <xacro:base
     length="${base_length}"
@@ -46,7 +46,7 @@
     radius="${wheel_radius}"
     width="${wheel_width}"
-    pos_x="${-wheel_pos_x}"
+    pos_x="${-wheel_pos_x_rear + base_link_x_offset_to_center}"
     pos_y="${wheel_pos_y}"
-    pos_z="${wheel_pos_z}"
+    pos_z="${wheel_pos_z + base_link_z_offset_to_center}"
     mass="${wheel_mass}"
   />
@@ -56,7 +56,7 @@
     radius="${wheel_radius}"
     width="${wheel_width}"
-    pos_x="${-wheel_pos_x}"
+    pos_x="${-wheel_pos_x_rear + base_link_x_offset_to_center}"
     pos_y="${-wheel_pos_y}"
-    pos_z="${wheel_pos_z}"
+    pos_z="${wheel_pos_z + base_link_z_offset_to_center}"
     mass="${wheel_mass}"
   />
@@ -64,7 +64,7 @@
     parent_link="base_link"
     side="front_left"
-    pos_x="${wheel_pos_x}"
+    pos_x="${wheel_pos_x_front + base_link_x_offset_to_center}"
     pos_y="${kingpin_width/2}"
-    pos_z="${wheel_pos_z}"
+    pos_z="${wheel_pos_z + base_link_z_offset_to_center}"
     mass="${wheel_mass_steering}"
     max_steer="${wheel_max_steer}"
@@ -73,37 +73,47 @@
     parent_link="base_link"
     side="front_right"
-    pos_x="${wheel_pos_x}"
+    pos_x="${wheel_pos_x_front + base_link_x_offset_to_center}"
     pos_y="${-kingpin_width/2}"
-    pos_z="${wheel_pos_z}"
+    pos_z="${wheel_pos_z + base_link_z_offset_to_center}"
     mass="${wheel_mass_steering}"
     max_steer="${wheel_max_steer}"
   />
-  <xacro:generic_laser>
+  <xacro:generic_laser
+    gz_laser_topic="scan"
+    gz_base_laser_topic="base_scan">
     <xacro:insert_block name="laser_pose" />
   </xacro:generic_laser>
-  <xacro:imu>
+  <xacro:imu
+    gz_imu_topic="ebot/imu/data"
+    gz_mag_topic="ebot/imu/mag">
     <xacro:insert_block name="imu_pose" />
   </xacro:imu>
+  <xacro:gps
+    gz_gps_topic="gps/fix">
+    <xacro:insert_block name="gps_pose"/>
+  </xacro:gps>
   <xacro:depth_sensor>
     <xacro:insert_block name="depth_sensor_pose" />
   </xacro:depth_sensor>
-  <xacro:hcsr04_sensor frame_id="hcsr04_back_left">
-    <xacro:insert_block name="range_back_left_pose" />
+  <xacro:hcsr04_sensor
+    frame_id="hcsr04_back_left"
+    parent_link="base_link">
+    <xacro:insert_block name="hcsr04_range_back_left_pose" />
   </xacro:hcsr04_sensor>
-  <xacro:hcsr04_sensor frame_id="hcsr04_back_right">
-    <xacro:insert_block name="range_back_right_pose" />
+  <xacro:hcsr04_sensor
+    frame_id="hcsr04_back_right"
+    parent_link="base_link">
+    <xacro:insert_block name="hcsr04_range_back_right_pose" />
   </xacro:hcsr04_sensor>
-  <xacro:depthai_camera
-   camera_name = "${depth_camera_name}"
-   parent = "${depth_parent_frame}"
-   camera_model = "${depth_camera_model}"
-   base_frame = "${depth_base_frame}"
-   cam_pos_x = "${depth_cam_pos_x}"
-   cam_pos_y = "${depth_cam_pos_y}"
-   cam_pos_z = "${depth_cam_pos_z}"
-   cam_roll = "${depth_cam_roll}"
-   cam_pitch = "${depth_cam_pitch}"
-   cam_yaw = "${depth_cam_yaw}"
-  />
+  <xacro:tof_sensor
+    frame_id="front_left_tof_frame"
+    parent_link="base_link">
+    <xacro:insert_block name="tof_sensor_front_left_pose" />
+  </xacro:tof_sensor>
+  <xacro:tof_sensor
+    frame_id="front_right_tof_frame"
+    parent_link="base_link">
+    <xacro:insert_block name="tof_sensor_front_right_pose" />
+  </xacro:tof_sensor>
   <gazebo>
     <plugin filename="gz-sim-joint-state-publisher-system" name="gz::sim::systems::JointStatePublisher"/>
@@ -111,6 +121,7 @@
       <render_engine>ogre2</render_engine>
     </plugin>
-    <plugin filename="gz-sim-imu-system" name="gz::sim::systems::Imu">
-    </plugin>
+    <plugin filename="gz-sim-imu-system" name="gz::sim::systems::Imu"/>
+    <plugin filename="gz-sim-magnetometer-system" name="gz::sim::systems::Magnetometer"/>
+    <plugin filename="gz-sim-navsat-system" name="gz::sim::systems::NavSat"/>
   </gazebo>
   <xacro:ackermann_drive_controller
@@ -120,4 +131,6 @@
     kingpin_width = "${kingpin_width}"
     wheel_radius = "${wheel_radius}"
+    gz_odom_topic="/ebot/odom"
+    gz_cmd_vel_topic="/cmd_vel/muxed"
   />
-  </robot>
+</robot>

Commit message: Fix Jeep TOF tilt

File: urdf/jeep_properties.urdf.xacro (robot description, xacro)
@@ -55,5 +55,5 @@
   <!-- Fix - check pitch angle and y offset -->
   <xacro:property name="tof_sensor_front_left_pose">
-    <origin xyz="${0.530 + base_link_x_offset_to_center} 0.013 ${0.095 + base_link_z_offset_to_center}" rpy="0 ${M_PI*12.0/180.0} ${M_PI*30.0/180.0}"/>
+    <origin xyz="${0.530 + base_link_x_offset_to_center} 0.013 ${0.095 + base_link_z_offset_to_center}" rpy="0 ${M_PI*14.0/180.0} ${M_PI*30.0/180.0}"/>
   </xacro:property>
   <xacro:property name="tof_sensor_front_right_pose">
